Commit message: 优化 Nav2 控制器参数并新增 Python 自动巡逻脚本

File: src/swarm_description/urdf/mobile_base.xacro (robot description, xacro)
@@ -66,6 +66,5 @@
             <gazebo reference="${prefix}_wheel_link">
                 <material>Gazebo/FlatBlack</material>
-                <mu1>1.0</mu1>
-                <mu2>1.0</mu2>
+                <mu1>1.0</mu1> <mu2>1.0</mu2>
             </gazebo>
         </xacro:macro>

File: src/swarm_description/urdf/robot.urdf.xacro (robot description, xacro)
@@ -13,14 +13,23 @@
             <wheel_separation>0.28</wheel_separation>
             <wheel_radius>0.045</wheel_radius>
-            <topic>cmd_vel</topic>
-            <odom_topic>odom</odom_topic>
+            <max_linear_acceleration>1</max_linear_acceleration>
+            <min_linear_acceleration>-1</min_linear_acceleration>
+            <max_angular_acceleration>2</max_angular_acceleration>
+            <min_angular_acceleration>-2</min_angular_acceleration>
+            <max_linear_velocity>0.5</max_linear_velocity>
+            <min_linear_velocity>-0.5</min_linear_velocity>
+            <max_angular_velocity>1</max_angular_velocity>
+            <min_angular_velocity>-1</min_angular_velocity>
+            <topic>cmd_vel</topic>       <odom_topic>odom</odom_topic> <tf_topic>/tf</tf_topic>
             <frame_id>odom</frame_id>
             <child_frame_id>base_footprint</child_frame_id>
-            <tf_topic>/tf</tf_topic>
+            <odom_publish_frequency>50</odom_publish_frequency>
         </plugin>
         <plugin filename="gz-sim-joint-state-publisher-system" name="gz::sim::systems::JointStatePublisher">
-            <topic>/joint_states</topic>
+            <topic>joint_states</topic>
+            <update_rate>50</update_rate>
+            <joint_name>left_wheel_joint</joint_name>
+            <joint_name>right_wheel_joint</joint_name>
         </plugin>
-        <plugin filename="gz-sim-imu-system" name="gz::sim::systems::Imu"></plugin>
     </gazebo>
 </robot>

File: src/swarm_description/urdf/sensors_stack.xacro (robot description, xacro)
@@ -22,5 +22,5 @@
             <parent link="${parent_link}"/>
             <child link="lidar_link"/>
-            <origin xyz="0.05 0 ${chassis_height}" rpy="0 0 0"/>
+            <origin xyz="0.05 0 ${chassis_height + 0.01}" rpy="0 0 0"/>
         </joint>
         <gazebo reference="lidar_link">
@@ -58,5 +58,11 @@
             <parent link="${parent_link}"/>
             <child link="camera_link"/>
-            <origin xyz="0.12 0 ${chassis_height + 0.05}" rpy="0 0 0"/>
+            <origin xyz="0.12 0 ${chassis_height + 0.01}" rpy="0 0 0"/>
+        </joint>
+        <link name="camera_link_optical"/>
+        <joint name="camera_optical_joint" type="fixed">
+            <parent link="camera_link"/>
+            <child link="camera_link_optical"/>
+            <origin xyz="0 0 0" rpy="-1.5707 0 -1.5707"/>
         </joint>
         <gazebo reference="camera_link">
@@ -66,6 +72,7 @@
                 <always_on>1</always_on>
                 <update_rate>10</update_rate>
-                <topic>/camera/image</topic> <frame_id>camera_link</frame_id>
-                <gz_frame_id>camera_link</gz_frame_id>
+                <topic>/camera/image</topic>
+                <frame_id>camera_link_optical</frame_id>
+                <gz_frame_id>camera_link_optical</gz_frame_id>
                 <camera>
                     <horizontal_fov>1.2</horizontal_fov>
@@ -78,6 +85,7 @@
                 <always_on>1</always_on>
                 <update_rate>10</update_rate>
-                <topic>/camera/depth_image</topic> <frame_id>camera_link</frame_id>
-                <gz_frame_id>camera_link</gz_frame_id>
+                <topic>/camera/depth_image</topic>
+                <frame_id>camera_link_optical</frame_id>
+                <gz_frame_id>camera_link_optical</gz_frame_id>
                 <camera>
                     <horizontal_fov>1.2</horizontal_fov>
@@ -93,5 +101,6 @@
         <joint name="imu_joint" type="fixed">
             <parent link="${parent_link}"/>
-            <child link="imu_link"/><origin xyz="0 0 0.05"/>
+            <child link="imu_link"/>
+            <origin xyz="0 0 0.05" rpy="0 0 0"/>
         </joint>
          <gazebo reference="imu_link">
