Commit message: Added ros_control

File: src/swarm_description/urdf/robot.urdf.xacro (robot description, xacro)
@@ -7,29 +7,28 @@
     <xacro:mobile_base parent_link="base_footprint"/>
     <xacro:sensor_stack parent_link="chassis_main" chassis_height="0.10"/>
+    <ros2_control name="GazeboSimSystem" type="system">
+        <hardware>
+            <plugin>gz_ros2_control/GazeboSimSystem</plugin>
+        </hardware>
+        <joint name="left_wheel_joint">
+            <command_interface name="velocity">
+                <param name="min">-10.0</param>
+                <param name="max">10.0</param>
+            </command_interface>
+            <state_interface name="position"/>
+            <state_interface name="velocity"/>
+        </joint>
+        <joint name="right_wheel_joint">
+            <command_interface name="velocity">
+                <param name="min">-10.0</param>
+                <param name="max">10.0</param>
+            </command_interface>
+            <state_interface name="position"/>
+            <state_interface name="velocity"/>
+        </joint>
+    </ros2_control>
     <gazebo>
-        <plugin filename="gz-sim-diff-drive-system" name="gz::sim::systems::DiffDrive">
-            <left_joint>left_wheel_joint</left_joint>
-            <right_joint>right_wheel_joint</right_joint>
-            <wheel_separation>0.28</wheel_separation>
-            <wheel_radius>0.045</wheel_radius>
-            <max_linear_acceleration>1</max_linear_acceleration>
-            <min_linear_acceleration>-1</min_linear_acceleration>
-            <max_angular_acceleration>2</max_angular_acceleration>
-            <min_angular_acceleration>-2</min_angular_acceleration>
-            <max_linear_velocity>0.5</max_linear_velocity>
-            <min_linear_velocity>-0.5</min_linear_velocity>
-            <max_angular_velocity>1</max_angular_velocity>
-            <min_angular_velocity>-1</min_angular_velocity>
-            <topic>cmd_vel</topic>       <odom_topic>odom</odom_topic> <tf_topic>/tf</tf_topic>
-            <frame_id>odom</frame_id>
-            <child_frame_id>base_footprint</child_frame_id>
-            <publish_odom_tf>false</publish_odom_tf>
-            <odom_publish_frequency>50</odom_publish_frequency>
-        </plugin>
-        <plugin filename="gz-sim-joint-state-publisher-system" name="gz::sim::systems::JointStatePublisher">
-            <topic>joint_states</topic>
-            <update_rate>50</update_rate>
-            <joint_name>left_wheel_joint</joint_name>
-            <joint_name>right_wheel_joint</joint_name>
+        <plugin filename="gz_ros2_control-system" name="gz_ros2_control::GazeboSimROS2ControlPlugin">
+            <parameters>$(find swarm_bringup)/config/controllers.yaml</parameters>
         </plugin>
     </gazebo>
