Commit message: 二维码识别功能

File: src/swarm_description/urdf/sensors_stack.xacro (robot description, xacro)
@@ -58,5 +58,5 @@
             <parent link="${parent_link}"/>
             <child link="camera_link"/>
-            <origin xyz="0.12 0 ${chassis_height + 0.01}" rpy="0 0 0"/>
+            <origin xyz="0.12 0 ${chassis_height + 0.09}" rpy="0 -0.26 0"/>
         </joint>
         <link name="camera_link_optical"/>
